File: hardware/step.kicad_sch (KiCad schematic)
At the start: 51 parts, among them J101 Conn_01x01, J102 Conn_01x01, J103 CORTEX-DEBUG, SW101 SW_Push, SW102 SW_Push, U101 ATSAMD51J, U102 TPS78433QWDRBRQ1, Y101 32k768

Commit message: Update parts library
Parts:
- C101: footprint Capacitor_SMD:C_0603_1608Metric -> V2_Capacitor_SMD:C_0603; symbol Device:C_Small -> V2_Device:C_0603_10u; Mouser (none) -> 810-C1608X6S1A106M
- C102, C103, C104, C105, C106, C109: footprint Capacitor_SMD:C_0603_1608Metric -> V2_Capacitor_SMD:C_0603; symbol Device:C_Small -> V2_Device:C_0603_0u1; Mouser (none) -> 810-CGA3E2X7R1H104MA
- C107, C108: footprint Capacitor_SMD:C_0603_1608Metric -> V2_Capacitor_SMD:C_0603; symbol Device:C_Small -> V2_Device:C_0603_18p; Mouser (none) -> 603-CC603JRNPO9BN180
- C110, C111: footprint Capacitor_SMD:C_0805_2012Metric -> V2_Capacitor_SMD:C_0603; symbol Device:C_Small -> V2_Device:C_0805_10u; Mouser (none) -> 810-C2012X5R1E106K; Rating (none) -> 25V
- D101: footprint LED_SMD:LED_0603_1608Metric -> V2_LED:LED_0603; symbol Device:LED_Small -> V2_Device:LED_0603_Orange; Mouser (none) -> 755-SML-D12M8WT86C
- ESD101: Mouser (none) -> 947-RCLAMP0582N.TCT
- FID101, FID102, FID103: value Fiducial -> Fiducial_Paste
- INFO102: value ORDER-NUMBER -> Order_Number
- J101, J102: value Conn_01x01 -> WAGO 2065-100
- J103: value CORTEX-DEBUG -> Cortex_Debug
- R101, R105: footprint Resistor_SMD:R_0603_1608Metric -> V2_Resistor_SMD:R_0603; symbol Device:R_Small -> V2_Device:R_0603_100k; Mouser (none) -> 71-CRCW0603100KFKEAC
- R102, R103: footprint Resistor_SMD:R_0603_1608Metric -> V2_Resistor_SMD:R_0603; symbol Device:R_Small -> V2_Device:R_0603_10k; Mouser (none) -> 71-CRCW060310K0FKEAC
- R104: footprint Resistor_SMD:R_0603_1608Metric -> V2_Resistor_SMD:R_0603; symbol Device:R_Small -> V2_Device:R_0603_330R; Mouser (none) -> 71-CRCW0603330RFKEAC
- SW101, SW102: value SW_Push -> SKSG; symbol Switch:SW_Push -> V2_Switch:SKSG; Mouser (none) -> 688-SKSGACE010
- TVS101: value SMAJ36CA -> SMBJ36CA; footprint Diode_SMD:D_SMA -> V2_Diode_SMD:D_SMB; symbol V2_Diode:SMAJ36CA -> V2_Diode:SMBJ36CA; Mouser (none) -> 652-SMBJ36CA-Q
- TVS102: footprint Diode_SMD:D_0603_1608Metric -> V2_Diode_SMD:D_0603; Mouser (none) -> 652-CG0603MLC-05LE
- U101: Mouser (none) -> 556-ATSAMD51J19AMU
- U102: Mouser (none) -> 595-TPS78433QWDRBRQ1
- Y101: symbol Device:Crystal_Small -> V2_Device:Crystal_3.2x1.5_32k768; Mouser (none) -> 815-ABS0716632.768KT
Other:
- moved on the sheet: FID101, FID102, FID103, J101, J102, TVS101

Commit message: Update parts
Parts:
- C101: Manufacturer (none) -> TDK; Product (none) -> C1608X6S1A106M080AC
- C102, C103, C104, C105, C106, C109: Manufacturer (none) -> TDK; Product (none) -> CGA3E2X7R1H104M080AA
- C107, C108: Manufacturer (none) -> YAGEO; Product (none) -> CC0603JRNPO9BN180
- C110, C111: footprint V2_Capacitor_SMD:C_0603 -> V2_Capacitor_SMD:C_0805; Manufacturer (none) -> TDK; Product (none) -> C2012X5R1E106K125AB
- D101: Manufacturer (none) -> ROHM Semiconductor; Product (none) -> SML-D12M8WT86C
- D102, D103: LCSC (none) -> C965555; Manufacturer (none) -> Worldsemi; Product (none) -> WS2812B-2020
- ESD101: Manufacturer (none) -> Semtech; Mouser 947-RCLAMP0582N.TCT -> 947-RCLAMP0582N.TCT; Product (none) -> RCLAMP0582N.TCT
- J101, J102: Manufacturer (none) -> WAGO; Product (none) -> 2065-100/998-403
- R101, R105: Manufacturer (none) -> Vishay; Product (none) -> CRCW0603100KFKEAC; Rating (none) -> 100mW
- R102, R103: Manufacturer (none) -> Vishay; Product (none) -> CRCW060310K0FKEAC; Rating (none) -> 100mW
- R104: Manufacturer (none) -> Vishay; Product (none) -> CRCW0603330RFKEAC; Rating (none) -> 100mW
- SW101, SW102: Manufacturer (none) -> Alps Alpine; Product (none) -> SKSGACE010
- TVS101: Manufacturer (none) -> Bourns; Product (none) -> SMBJ36CA-Q; Rating (none) -> 36V
- TVS102: Manufacturer (none) -> Bourns; Product (none) -> CG0603MLC-05LE; Rating (none) -> 5V
- U101: Manufacturer (none) -> Microchip Technology; Mouser 556-ATSAMD51J19AMU -> 556-ATSAMD51J19AMU; Product (none) -> ATSAMD51J19A-MU
- U102: Manufacturer (none) -> Texas Instruments; Mouser 595-TPS78433QWDRBRQ1 -> 595-TPS78433QWDRBRQ1; Product (none) -> TPS78433QWDRBRQ1
- Y101: Manufacturer (none) -> ABRACON; Product (none) -> ABS07-166-32.768KHZ-T

Commit message: Refresh
Parts:
- C101: Rating (none) -> 10V
- C102, C103, C104, C105, C106, C109: Rating (none) -> 50V
- D101: Mouser 755-SML-D12M8WT86C -> 755-SML-D12D1WT86; Product SML-D12M8WT86C -> SML-D12D1WT86
- TVS101: value SMBJ36CA -> SMBJ33CA; symbol V2_Diode:SMBJ36CA -> V2_Diode:SMBJ33CA; Mouser 652-SMBJ36CA-Q -> 652-SMBJ33CA-Q; Product SMBJ36CA-Q -> SMBJ33CA-Q; Rating 36V -> 33V
Connections:
- net +24V renamed +28V

Commit message: Update library
Parts:
- J103: value Cortex_Debug -> Cortex; footprint V2_Cortex_Debug:Cortex_Debug_Pad -> V2_Connector_Debug:Cortex; symbol V2_Cortex_Debug:Cortex_Debug -> V2_Connector_Debug:Cortex
Changed lines of the file:
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@@
 		(at 237.49 144.78 0)
 		(unit 1)
-		(exclude_from_sim no)
+		(exclude_from_sim yes)
 		(in_bom no)
 		(on_board yes)
@@
 		(at 184.15 193.04 0)
 		(unit 1)
-		(exclude_from_sim no)
+		(exclude_from_sim yes)
 		(in_bom no)
 		(on_board yes)
@@
 		(at 184.15 172.72 0)
 		(unit 1)
-		(exclude_from_sim no)
+		(exclude_from_sim yes)
 		(in_bom no)
 		(on_board yes)
@@
 		(at 210.82 163.83 0)
 		(unit 1)
-		(exclude_from_sim no)
+		(exclude_from_sim yes)
 		(in_bom no)
 		(on_board yes)
@@
 		(at 256.54 176.53 0)
 		(unit 1)
-		(exclude_from_sim no)
+		(exclude_from_sim yes)
 		(in_bom no)
 		(on_board yes)
@@
 		(at 199.39 144.78 0)
 		(unit 1)
-		(exclude_from_sim no)
+		(exclude_from_sim yes)
 		(in_bom no)
 		(on_board yes)
@@
 	)
 	(symbol
-		(lib_id "V2_Cortex_Debug:Cortex_Debug")
+		(lib_id "V2_Connector_Debug:Cortex")
 		(at 120.65 107.95 0)
 		(unit 1)
@@
 		(dnp no)
 		(property "Reference" "J103"
-			(at 121.92 95.25 0)
+			(at 114.3 96.012 0)
 			(effects
 				(font
@@
 			)
 		)
-		(property "Value" "Cortex_Debug"
-			(at 121.92 97.79 0)
+		(property "Value" "Cortex"
+			(at 111.76 99.06 0)
 			(effects
 				(font
 					(size 1.27 1.27)
 				)
+				(justify left bottom)
 			)
 		)
-		(property "Footprint" "V2_Cortex_Debug:Cortex_Debug_Pad"
+		(property "Footprint" "V2_Connector_Debug:Cortex"
 			(at 120.65 121.92 0)
 			(effects
@@
 		(at 184.15 152.4 0)
 		(unit 1)
-		(exclude_from_sim no)
+		(exclude_from_sim yes)
 		(in_bom no)
 		(on_board yes)
@@
 		(at 184.15 182.88 0)
 		(unit 1)
-		(exclude_from_sim no)
+		(exclude_from_sim yes)
 		(in_bom no)
 		(on_board yes)
@@
 		(at 233.68 160.02 0)
 		(unit 1)
-		(exclude_from_sim no)
+		(exclude_from_sim yes)
 		(in_bom no)
 		(on_board yes)
@@
 	(symbol
 		(lib_id "V2_power:PWR_FLAG")
-		(at 251.46 21.59 90)
+		(at 251.46 21.59 0)
 		(unit 1)
 		(exclude_from_sim no)
@@
 		(dnp no)
 		(property "Reference" "#FLG0101"
-			(at 249.555 21.59 0)
+			(at 251.46 19.685 0)
 			(effects
 				(font
@@
 		)
 		(property "Value" "PWR_FLAG"
-			(at 242.57 21.59 90)
+			(at 242.316 21.59 0)
 			(effects
 				(font
@@
 		(at 184.15 162.56 0)
 		(unit 1)
-		(exclude_from_sim no)
+		(exclude_from_sim yes)
 		(in_bom no)
 		(on_board yes)
@@
 		(at 162.56 173.99 0)
 		(unit 1)
-		(exclude_from_sim no)
+		(exclude_from_sim yes)
 		(in_bom no)
 		(on_board yes)
@@
 		(at 220.98 144.78 0)
 		(unit 1)
-		(exclude_from_sim no)
+		(exclude_from_sim yes)
 		(in_bom no)
 		(on_board yes)
@@
 		(at 256.54 165.1 0)
 		(unit 1)
-		(exclude_from_sim no)
+		(exclude_from_sim yes)
 		(in_bom no)
 		(on_board yes)
@@
 		(at 256.54 153.67 0)
 		(unit 1)
-		(exclude_from_sim no)
+		(exclude_from_sim yes)
 		(in_bom no)
 		(on_board yes)
@@
 		(at 163.195 160.02 0)
 		(unit 1)
-		(exclude_from_sim no)
+		(exclude_from_sim yes)
 		(in_bom no)
 		(on_board yes)
@@
 		(at 233.68 175.26 0)
 		(unit 1)
-		(exclude_from_sim no)
+		(exclude_from_sim yes)
 		(in_bom no)
 		(on_board yes)

Commit message: Replace Order_Number
Parts:
- H101, H103, H105, H107, H108: value MountingHole_2mm -> 2mm
- H102, H104, H106: value MountingHole_3mm -> 3mm
- INFO102: value Order_Number -> (none); footprint V2_Production:Order_Number -> V2_Production:Revision; symbol V2_Production:Order_Number -> V2_Production:Revision
Other:
- moved on the sheet: FID101, FID102, FID103, H101, H102, H103, H104, H105, H106, H107, H108, ICON101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

Commit message: Update Library
Parts:
- C101: symbol V2_Device:C_0603_10u -> V2_Capacitor:0603_10u
- C102, C103, C104, C105, C106, C109: symbol V2_Device:C_0603_0u1 -> V2_Capacitor:0603_0u1
- C107, C108: symbol V2_Device:C_0603_18p -> V2_Capacitor:0603_18p
- C110, C111: symbol V2_Device:C_0805_10u -> V2_Capacitor:0805_10u
- D101: symbol V2_Device:LED_0603_Orange -> V2_LED:0603_Orange
- INFO102: value (none) -> ~
- R101, R105: symbol V2_Device:R_0603_100k -> V2_Resistor:0603_100k
- R102, R103: symbol V2_Device:R_0603_10k -> V2_Resistor:0603_10k
- R104: symbol V2_Device:R_0603_330R -> V2_Resistor:0603_330R
- Y101: symbol V2_Device:Crystal_3.2x1.5_32k768 -> V2_Crystal:3.2x1.5_32k768

Commit message: Update
Changed lines of the file:
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@@
 		)
 		(property "Value" "+5V"
-			(at 184.15 121.92 90)
+			(at 185.166 121.92 90)
 			(effects
 				(font
 					(size 1.27 1.27)
+					(color 255 92 187 1)
 				)
 			)
@@
 				(font
 					(size 1.27 1.27)
+					(color 255 92 187 1)
 				)
 			)
@@
 		(at 223.52 165.1 0)
 		(unit 1)
-		(exclude_from_sim no)
+		(exclude_from_sim yes)
 		(in_bom no)
 		(on_board yes)
@@
 			)
 		)
-		(property "Sim.Enable" "0"
-			(at 223.52 165.1 0)
-			(effects
-				(font
-					(size 1.27 1.27)
-				)
-				(hide yes)
-			)
-		)
 		(instances
 			(project ""
@@
 				(font
 					(size 1.27 1.27)
+					(color 255 92 187 1)
 				)
 			)
@@
 		(on_board yes)
 		(dnp no)
-		(fields_autoplaced yes)
 		(property "Reference" "#PWR105"
 			(at 243.84 31.75 0)
@@
 		)
 		(property "Value" "+28V"
-			(at 236.22 31.7499 90)
+			(at 233.172 31.7499 90)
 			(effects
 				(font
 					(size 1.27 1.27)
+					(color 255 92 187 1)
 				)
-				(justify left)
 			)
 		)
@@
 				(font
 					(size 1.27 1.27)
+					(color 255 92 187 1)
 				)
 			)
@@
 		(at 190.5 152.4 0)
 		(unit 1)
-		(exclude_from_sim no)
+		(exclude_from_sim yes)
 		(in_bom no)
 		(on_board yes)
@@
 			)
 		)
-		(property "Sim.Enable" "0"
-			(at 190.5 152.4 0)
-			(effects
-				(font
-					(size 1.27 1.27)
-				)
-				(hide yes)
-			)
-		)
 		(instances
 			(project "pulse"
@@
 		(on_board yes)
 		(dnp no)
-		(fields_autoplaced yes)
 		(property "Reference" "#PWR102"
 			(at 252.73 19.05 0)
@@
 		)
 		(property "Value" "+28V"
-			(at 260.35 19.0499 90)
+			(at 264.414 19.0499 90)
 			(effects
 				(font
 					(size 1.27 1.27)
+					(color 255 92 187 1)
 				)
-				(justify left)
 			)
 		)
@@
 		)
 		(property "Value" "+3V3"
-			(at 72.39 17.78 0)
+			(at 72.39 17.018 0)
 			(effects
 				(font
 					(size 1.27 1.27)
+					(color 255 92 187 1)
 				)
 			)
@@
 				(font
 					(size 1.27 1.27)
+					(color 255 92 187 1)
 				)
 			)
@@
 		)
 		(property "Value" "+3V3"
-			(at 41.91 121.92 90)
+			(at 41.148 121.92 90)
 			(effects
 				(font
 					(size 1.27 1.27)
+					(color 255 92 187 1)
 				)
 			)
@@
 		(at 223.52 152.4 0)
 		(unit 1)
-		(exclude_from_sim no)
+		(exclude_from_sim yes)
 		(in_bom no)
 		(on_board yes)
@@
 			)
 		)
-		(property "Sim.Enable" "0"
-			(at 223.52 152.4 0)
-			(effects
-				(font
-					(size 1.27 1.27)
-				)
-				(hide yes)
-			)
-		)
 		(instances
 			(project "pulse"
@@
 				(font
 					(size 1.27 1.27)
+					(color 255 92 187 1)
 				)
 			)
@@
 				(font
 					(size 1.27 1.27)
+					(color 255 92 187 1)
 				)
 			)
@@
 		)
 		(property "Value" "+3V3"
-			(at 46.99 46.99 90)
+			(at 46.482 48.26 90)
 			(effects
 				(font
 					(size 1.27 1.27)
+					(color 255 92 187 1)
 				)
-				(justify bottom)
 			)
 		)
@@
 		)
 		(property "Value" "+3V3"
-			(at 102.87 102.87 90)
+			(at 101.854 102.87 90)
 			(effects
 				(font
 					(size 1.27 1.27)
+					(color 255 92 187 1)
 				)
 			)
@@
 		(at 190.5 160.02 0)
 		(unit 1)
-		(exclude_from_sim no)
+		(exclude_from_sim yes)
 		(in_bom no)
 		(on_board yes)
@@
 			)
 		)
-		(property "Sim.Enable" "0"
-			(at 190.5 160.02 0)
-			(effects
-				(font
-					(size 1.27 1.27)
-				)
-				(hide yes)
-			)
-		)
 		(instances
 			(project "pulse"
@@
 		(at 157.48 160.02 0)
 		(unit 1)
-		(exclude_from_sim no)
+		(exclude_from_sim yes)
 		(in_bom no)
 		(on_board yes)
@@
 			)
 		)
-		(property "Sim.Enable" "0"
-			(at 157.48 160.02 0)
-			(effects
-				(font
-					(size 1.27 1.27)
-				)
-				(hide yes)
-			)
-		)
 		(instances
 			(project ""
@@
 		(at 223.52 158.75 0)
 		(unit 1)
-		(exclude_from_sim no)
+		(exclude_from_sim yes)
 		(in_bom no)
 		(on_board yes)
@@
 			)
 		)
-		(property "Sim.Enable" "0"
-			(at 223.52 158.75 0)
-			(effects
-				(font
-					(size 1.27 1.27)
-				)
-				(hide yes)
-			)
-		)
 		(instances
 			(project ""
@@
 		(at 190.5 168.91 0)
 		(unit 1)
-		(exclude_from_sim no)
+		(exclude_from_sim yes)
 		(in_bom no)
 		(on_board yes)
@@
 			(at 190.5 168.91 0)
 			(effects
-				(font
-					(size 1.27 1.27)
-				)
-				(hide yes)
-			)
-		)
-		(property "Sim.Enable" "0"
-			(at 190.5 168.91 0)
-			(effects
