File: hardware/step.kicad_sch (KiCad schematic)
At the start: 51 parts, among them J101 Cortex, J102 WAGO 2065-100, J103 WAGO 2065-100, SW101 SKSG, SW102 SKSG, U101 TPS78433QWDRBRQ1, U102 ATSAMD51J, Y101 32k768

Commit message: Rename
Connections:
- net +5V: now also U101.6 (EN)
Other:
- sheet Link Plug: file LinkPlug.kicad_sch -> Link-Plug.kicad_sch
- sheet Link Socket: file LinkSocket.kicad_sch -> Link-Socket.kicad_sch
- sheet Stepper-1: file StepperDriver.kicad_sch -> Stepper.kicad_sch
- sheet Stepper-2: file StepperDriver.kicad_sch -> Stepper.kicad_sch
- sheet Stepper-3: file StepperDriver.kicad_sch -> Stepper.kicad_sch
- sheet Stepper-4: file StepperDriver.kicad_sch -> Stepper.kicad_sch
Changed lines of the file:
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@@
 	(title_block
 		(title "V2 step")
-		(date "2026-07-31")
+		(date "2026-08-30")
 		(rev "2026-05-26")
 		(company "Versio Duo")
@@
 		(unit 1)
 		(body_style 1)
-		(exclude_from_sim no)
+		(exclude_from_sim yes)
 		(in_bom no)
 		(on_board yes)
@@
 			)
 		)
-		(property "Sim.Enable" "0"
-			(at 223.52 165.1 0)
-			(hide yes)
-			(show_name no)
-			(do_not_autoplace no)
-			(effects
-				(font
-					(size 1.27 1.27)
-				)
-			)
-		)
 		(instances
 			(project "step"
@@
 		(unit 1)
 		(body_style 1)
-		(exclude_from_sim no)
+		(exclude_from_sim yes)
 		(in_bom no)
 		(on_board yes)
@@
 			)
 		)
-		(property "Sim.Enable" "0"
-			(at 190.5 152.4 0)
-			(hide yes)
-			(show_name no)
-			(do_not_autoplace no)
-			(effects
-				(font
-					(size 1.27 1.27)
-				)
-			)
-		)
 		(instances
 			(project "step"
@@
 		(unit 1)
 		(body_style 1)
-		(exclude_from_sim no)
+		(exclude_from_sim yes)
 		(in_bom no)
 		(on_board yes)
@@
 			)
 		)
-		(property "Sim.Enable" "0"
-			(at 223.52 152.4 0)
-			(hide yes)
-			(show_name no)
-			(do_not_autoplace no)
-			(effects
-				(font
-					(size 1.27 1.27)
-				)
-			)
-		)
 		(instances
 			(project "step"
@@
 		(unit 1)
 		(body_style 1)
-		(exclude_from_sim no)
+		(exclude_from_sim yes)
 		(in_bom no)
 		(on_board yes)
@@
 			)
 		)
-		(property "Sim.Enable" "0"
-			(at 190.5 160.02 0)
-			(hide yes)
-			(show_name no)
-			(do_not_autoplace no)
-			(effects
-				(font
-					(size 1.27 1.27)
-				)
-			)
-		)
 		(instances
 			(project "step"
@@
 		(unit 1)
 		(body_style 1)
-		(exclude_from_sim no)
+		(exclude_from_sim yes)
 		(in_bom no)
 		(on_board yes)
@@
 			)
 		)
-		(property "Sim.Enable" "0"
-			(at 157.48 160.02 0)
-			(hide yes)
-			(show_name no)
-			(do_not_autoplace no)
-			(effects
-				(font
-					(size 1.27 1.27)
-				)
-			)
-		)
 		(instances
 			(project "step"
@@
 		(unit 1)
 		(body_style 1)
-		(exclude_from_sim no)
+		(exclude_from_sim yes)
 		(in_bom no)
 		(on_board yes)
@@
 			)
 		)
-		(property "Sim.Enable" "0"
-			(at 223.52 158.75 0)
-			(hide yes)
-			(show_name no)
-			(do_not_autoplace no)
-			(effects
-				(font
-					(size 1.27 1.27)
-				)
-			)
-		)
 		(instances
 			(project "step"
@@
 		(unit 1)
 		(body_style 1)
-		(exclude_from_sim no)
+		(exclude_from_sim yes)
 		(in_bom no)
 		(on_board yes)
@@
 			)
 		)
-		(property "Sim.Enable" "0"
-			(at 190.5 168.91 0)
-			(hide yes)
-			(show_name no)
-			(do_not_autoplace no)
-			(effects
-				(font
-					(size 1.27 1.27)
-				)
-			)
-		)
 		(instances
 			(project "step"
@@
 			)
 		)
-		(property "Sheetfile" "LinkSocket.kicad_sch"
+		(property "Sheetfile" "Link-Socket.kicad_sch"
 			(at 266.7 128.8546 0)
 			(hide yes)
@@
 			)
 		)
-		(property "Sheetfile" "StepperDriver.kicad_sch"
+		(property "Sheetfile" "Stepper.kicad_sch"
 			(at 205.74 85.6746 0)
 			(hide yes)
@@
 			)
 		)
-		(property "Sheetfile" "StepperDriver.kicad_sch"
+		(property "Sheetfile" "Stepper.kicad_sch"
 			(at 170.18 51.3846 0)
 			(hide yes)
@@
 			)
 		)
-		(property "Sheetfile" "StepperDriver.kicad_sch"
+		(property "Sheetfile" "Stepper.kicad_sch"
 			(at 205.74 51.3846 0)
 			(hide yes)
@@
 			)
 		)
-		(property "Sheetfile" "StepperDriver.kicad_sch"
+		(property "Sheetfile" "Stepper.kicad_sch"
 			(at 170.18 85.6746 0)
 			(hide yes)
@@
 			)
 		)
-		(property "Sheetfile" "LinkPlug.kicad_sch"
+		(property "Sheetfile" "Link-Plug.kicad_sch"
 			(at 227.33 123.7746 0)
 			(hide yes)
