File: hardware/LinkSocket.kicad_sch (KiCad schematic)
At the start: 4 parts, among them J2001 2x05_Horizontal, U2001 THVD24x2

Commit message: Update parts library
Parts:
- C2001: footprint Capacitor_SMD:C_0603_1608Metric -> V2_Capacitor_SMD:C_0603; symbol Device:C_Small -> V2_Device:C_0603_0u1; Mouser (none) -> 810-CGA3E2X7R1H104MA
- J2001: Mouser (none) -> 649-200211120001T4LF
- R2001: footprint Resistor_SMD:R_0603_1608Metric -> V2_Resistor_SMD:R_0603; symbol Device:R_Small -> V2_Device:R_0603_100R; Mouser (none) -> 71-CRCW0603100RFKEAH
- U2001: value THVD24x2 -> THVD2442; symbol V2_Interface_RS485:THVD24x2 -> V2_Interface_RS485:THVD2442; Mouser (none) -> 595-THVD2442DRCR
Other:
- moved on the sheet: C2001, J2001, R2001, U2001

Commit message: Update parts
Parts:
- C2001: Manufacturer (none) -> TDK; Product (none) -> CGA3E2X7R1H104M080AA
- J2001: Manufacturer (none) -> Amphenol FCI; Product (none) -> 20021112-00010T4LF
- R2001: Manufacturer (none) -> Vishay; Product (none) -> CRCW0603100RFKEAHP; Rating (none) -> 330mW
- U2001: Manufacturer (none) -> Texas Instruments; Mouser 595-THVD2442DRCR -> 595-THVD2442DRCR; Product (none) -> THVD2442DRCR
Changed lines of the file:
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@@
 			)
 		)
-		(property "Mouser" " 595-THVD2442DRCR "
+		(property "Mouser" "595-THVD2442DRCR"
+			(at 151.13 85.09 0)
+			(effects
+				(font
+					(size 1.27 1.27)
+				)
+				(hide yes)
+			)
+		)
+		(property "Product" "THVD2442DRCR "
+			(at 151.13 118.11 0)
+			(effects
+				(font
+					(size 1.27 1.27)
+				)
+				(hide yes)
+			)
+		)
+		(property "Manufacturer" "Texas Instruments"
+			(at 151.13 115.57 0)
+			(effects
+				(font
+					(size 1.27 1.27)
+				)
+				(hide yes)
+			)
+		)
+		(property "Sim.Enable" ""
 			(at 151.13 85.09 0)
 			(effects
@@
 			)
 		)
+		(property "Rating" "330mW"
+			(at 162.56 102.87 0)
+			(effects
+				(font
+					(size 1.27 1.27)
+				)
+				(hide yes)
+			)
+		)
+		(property "Manufacturer" "Vishay"
+			(at 162.56 97.79 0)
+			(effects
+				(font
+					(size 1.27 1.27)
+				)
+				(hide yes)
+			)
+		)
+		(property "Product" "CRCW0603100RFKEAHP"
+			(at 162.56 100.33 0)
+			(effects
+				(font
+					(size 1.27 1.27)
+				)
+				(hide yes)
+			)
+		)
+		(property "Sim.Enable" ""
+			(at 162.56 80.01 0)
+			(effects
+				(font
+					(size 1.27 1.27)
+				)
+				(hide yes)
+			)
+		)
 		(pin "1"
 		)
@@
 			)
 		)
+		(property "Manufacturer" "Amphenol FCI"
+			(at 151.13 162.56 0)
+			(effects
+				(font
+					(size 1.27 1.27)
+				)
+				(hide yes)
+			)
+		)
+		(property "Product" "20021112-00010T4LF"
+			(at 151.13 165.1 0)
+			(effects
+				(font
+					(size 1.27 1.27)
+				)
+				(hide yes)
+			)
+		)
+		(property "Sim.Enable" ""
+			(at 151.13 144.78 0)
+			(effects
+				(font
+					(size 1.27 1.27)
+				)
+				(hide yes)
+			)
+		)
 		(pin "1"
 		)
@@
 			(effects
 				(font
+					(size 1.27 1.27)
+				)
+				(hide yes)
+			)
+		)
+		(property "Manufacturer" "TDK"
+			(at 172.72 80.01 0)
+			(effects
+				(font
+					(size 1.27 1.27)
+				)
+				(hide yes)
+			)
+		)
+		(property "Product" "CGA3E2X7R1H104M080AA"
+			(at 172.72 82.55 0)
+			(effects
+				(font
+					(size 1.27 1.27)
+				)
+				(hide yes)
+			)
+		)
+		(property "Sim.Enable" ""
+			(at 172.72 64.77 0)
+			(effects
+				(font

Commit message: Refresh
Parts:
- C2001: Rating (none) -> 50V
Changed lines of the file:
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@@
 			)
 		)
-		(property "Description" "Power symbol creates a global label with name \"+3V3\""
+		(property "Description" ""
 			(at 151.13 62.23 0)
 			(effects
@@
 			)
 		)
-		(property "Sim.Enable" ""
-			(at 151.13 85.09 0)
-			(effects
-				(font
-					(size 1.27 1.27)
-				)
-				(hide yes)
-			)
-		)
 		(pin "1"
 		)
@@
 			)
 		)
-		(property "Description" "Power symbol creates a global label with name \"GND\" , ground"
+		(property "Description" ""
 			(at 144.78 142.24 0)
 			(effects
@@
 			)
 		)
-		(property "Description" "Power symbol creates a global label with name \"GND\" , ground"
+		(property "Description" ""
 			(at 151.13 100.33 0)
 			(effects
@@
 			)
 		)
-		(property "Description" "Power symbol creates a global label with name \"GND\" , ground"
+		(property "Description" ""
 			(at 172.72 67.31 0)
 			(effects
@@
 			)
 		)
-		(property "Sim.Enable" ""
-			(at 162.56 80.01 0)
-			(effects
-				(font
-					(size 1.27 1.27)
-				)
-				(hide yes)
-			)
-		)
 		(pin "1"
 		)
@@
 			)
 		)
-		(property "Description" "Power symbol creates a global label with name \"GND\" , ground"
+		(property "Description" ""
 			(at 157.48 147.32 0)
 			(effects
@@
 			)
 		)
-		(property "Sim.Enable" ""
-			(at 151.13 144.78 0)
-			(effects
-				(font
-					(size 1.27 1.27)
-				)
-				(hide yes)
-			)
-		)
 		(pin "1"
 		)
@@
 			)
 		)
-		(property "Sim.Enable" ""
-			(at 172.72 64.77 0)
+		(property "Rating" "50V"
+			(at 172.72 87.63 0)
 			(effects
 				(font
@@
 			)
 		)
-		(property "Description" "Power symbol creates a global label with name \"+5V\""
+		(property "Description" ""
 			(at 144.78 147.32 0)
 			(effects
@@
 			)
 		)
-		(property "Description" "Power symbol creates a global label with name \"+5V\""
+		(property "Description" ""
 			(at 157.48 142.24 0)
 			(effects

Commit message: Update Library
Parts:
- C2001: symbol V2_Device:C_0603_0u1 -> V2_Capacitor:0603_0u1
- R2001: symbol V2_Device:R_0603_100R -> V2_Resistor:0603_100R
Changed lines of the file:
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@@
 		(on_board yes)
 		(dnp no)
-		(property "Reference" "#PWR02001"
+		(property "Reference" "#PWR2001"
 			(at 151.13 66.04 0)
 			(effects
@@
 			(project "pulse"
 				(path "/6c8448b4-b04d-47e1-934e-e40cbe27a7be/2a03ea79-269e-4abf-833c-000ba0ff13d7"
-					(reference "#PWR02001")
+					(reference "#PWR2001")
 					(unit 1)
 				)
@@
 		(on_board yes)
 		(dnp no)
-		(property "Reference" "#PWR02004"
+		(property "Reference" "#PWR2004"
 			(at 138.43 142.24 0)
 			(effects
@@
 			(project "pulse"
 				(path "/6c8448b4-b04d-47e1-934e-e40cbe27a7be/2a03ea79-269e-4abf-833c-000ba0ff13d7"
-					(reference "#PWR02004")
+					(reference "#PWR2004")
 					(unit 1)
 				)
@@
 		(on_board yes)
 		(dnp no)
-		(property "Reference" "#PWR02003"
+		(property "Reference" "#PWR2003"
 			(at 151.13 106.68 0)
 			(effects
@@
 			(project "pulse"
 				(path "/6c8448b4-b04d-47e1-934e-e40cbe27a7be/2a03ea79-269e-4abf-833c-000ba0ff13d7"
-					(reference "#PWR02003")
+					(reference "#PWR2003")
 					(unit 1)
 				)
@@
 		(on_board yes)
 		(dnp no)
-		(property "Reference" "#PWR02002"
+		(property "Reference" "#PWR2002"
 			(at 172.72 73.66 0)
 			(effects
@@
 			(project "pulse"
 				(path "/6c8448b4-b04d-47e1-934e-e40cbe27a7be/2a03ea79-269e-4abf-833c-000ba0ff13d7"
-					(reference "#PWR02002")
-					(unit 1)
-				)
-			)
-		)
-	)
-	(symbol
-		(lib_id "V2_Device:R_0603_100R")
+					(reference "#PWR2002")
+					(unit 1)
+				)
+			)
+		)
+	)
+	(symbol
+		(lib_id "V2_Resistor:0603_100R")
 		(at 162.56 80.01 0)
 		(unit 1)
@@
 		(on_board yes)
 		(dnp no)
-		(property "Reference" "#PWR02007"
+		(property "Reference" "#PWR2007"
 			(at 163.83 147.32 0)
 			(effects
@@
 			(project "pulse"
 				(path "/6c8448b4-b04d-47e1-934e-e40cbe27a7be/2a03ea79-269e-4abf-833c-000ba0ff13d7"
-					(reference "#PWR02007")
+					(reference "#PWR2007")
 					(unit 1)
 				)
@@
 	)
 	(symbol
-		(lib_id "V2_Device:C_0603_0u1")
+		(lib_id "V2_Capacitor:0603_0u1")
 		(at 172.72 64.77 0)
 		(unit 1)
@@
 		(on_board yes)
 		(dnp no)
-		(property "Reference" "#PWR02006"
+		(property "Reference" "#PWR2006"
 			(at 148.59 147.32 0)
 			(effects
@@
 			(project "pulse"
 				(path "/6c8448b4-b04d-47e1-934e-e40cbe27a7be/2a03ea79-269e-4abf-833c-000ba0ff13d7"
-					(reference "#PWR02006")
+					(reference "#PWR2006")
 					(unit 1)
 				)
@@
 		(on_board yes)
 		(dnp no)
-		(property "Reference" "#PWR02005"
+		(property "Reference" "#PWR2005"
 			(at 153.67 142.24 0)
 			(effects
@@
 			(project "pulse"
 				(path "/6c8448b4-b04d-47e1-934e-e40cbe27a7be/2a03ea79-269e-4abf-833c-000ba0ff13d7"
-					(reference "#PWR02005")
-					(unit 1)
-				)
+					(reference "#PWR2005")
+					(unit 1)
+				)

Commit message: Update
Changed lines of the file:
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@@
 		)
 		(property "Value" "+3V3"
-			(at 151.13 58.42 0)
-			(effects
-				(font
-					(size 1.27 1.27)
+			(at 151.13 57.912 0)
+			(effects
+				(font
+					(size 1.27 1.27)
+					(color 255 92 187 1)
 				)
 			)
@@
 		)
 		(property "Value" "+5V"
-			(at 139.7 147.32 90)
-			(effects
-				(font
-					(size 1.27 1.27)
+			(at 138.938 147.32 90)
+			(effects
+				(font
+					(size 1.27 1.27)
+					(color 255 92 187 1)
 				)
 			)
@@
 		)
 		(property "Value" "+5V"
-			(at 162.56 142.24 90)
-			(effects
-				(font
-					(size 1.27 1.27)
-				)
-			)
+			(at 163.322 142.24 90)
+			(effects
+				(font
+					(size 1.27 1.27)
+					(color 255 92 187 1)
+				)
+			)

Commit message: KiCad 10
Other:
- company: Socket -> Versio Duo
