File: hardware/LinkSocket.kicad_sch (KiCad schematic)
At the start: 4 parts, among them J2001 2x05_Horizontal, U2001 THVD2442

Commit message: Update
Parts:
- C2001: Id (none) -> Capacitor:${SYMBOL_NAME}
- J2001: Id (none) -> Header:${SYMBOL_NAME}
- R2001: Id (none) -> Resistor:${SYMBOL_NAME}
- U2001: Id (none) -> RS485:${SYMBOL_NAME}; Rating (none) -> 20Mbps
Other:
- title: V2 Link -> V2 step
Changed lines of the file:
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@@
 	(paper "A4")
 	(title_block
-		(title "V2 Link")
-		(date "2026-03-20")
+		(title "V2 step")
+		(date "2026-04-11")
 		(rev "2026-02-10")
 		(company "Versio Duo")
+		(comment 1 "Stepper Motor Controller")
 	)
 	(junction
@@
 			)
 		)
+		(property "Id" "RS485:${SYMBOL_NAME}"
+			(at 151.13 116.84 0)
+			(hide yes)
+			(show_name no)
+			(do_not_autoplace no)
+			(effects
+				(font
+					(size 1.27 1.27)
+				)
+			)
+		)
+		(property "Rating" "20Mbps"
+			(at 152.4 124.46 0)
+			(hide yes)
+			(show_name no)
+			(do_not_autoplace no)
+			(effects
+				(font
+					(size 1.27 1.27)
+				)
+			)
+		)
 		(pin "1"
 		)
@@
 			)
 		)
+		(property "Id" "Resistor:${SYMBOL_NAME}"
+			(at 162.56 93.98 0)
+			(hide yes)
+			(show_name no)
+			(do_not_autoplace no)
+			(effects
+				(font
+					(size 1.27 1.27)
+				)
+			)
+		)
 		(pin "1"
 		)
@@
 			)
 		)
+		(property "Id" "Header:${SYMBOL_NAME}"
+			(at 151.13 160.02 0)
+			(hide yes)
+			(show_name no)
+			(do_not_autoplace no)
+			(effects
+				(font
+					(size 1.27 1.27)
+				)
+			)
+		)
 		(pin "1"
 		)
@@
 			(hide yes)
 			(show_name no)
+			(do_not_autoplace no)
+			(effects
+				(font
+					(size 1.27 1.27)
+				)
+			)
+		)
+		(property "Id" "Capacitor:${SYMBOL_NAME}"
+			(at 172.72 80.01 0)
+			(hide yes)
+			(show_name no)

Commit message: Update
Parts:
- J2001: Rating (none) -> 1A
Changed lines of the file:
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@@
 	(title_block
 		(title "V2 step")
-		(date "2026-04-11")
+		(date "2026-04-14")
 		(rev "2026-02-10")
 		(company "Versio Duo")
@@
 			(hide yes)
 			(show_name no)
+			(do_not_autoplace no)
+			(effects
+				(font
+					(size 1.27 1.27)
+				)
+			)
+		)
+		(property "Rating" "1A"
+			(at 151.13 175.26 0)
+			(hide yes)
+			(show_name no)

Commit message: Good Bye Imperial
Parts:
- C2001: footprint V2_Capacitor_SMD:C_0603 -> V2_Capacitor_SMD:C_1608; symbol V2_Capacitor:0603_0u1 -> V2_Capacitor:1608_0u1
- R2001: footprint V2_Resistor_SMD:R_0603 -> V2_Resistor_SMD:R_1608; symbol V2_Resistor:0603_100R -> V2_Resistor:1608_100R
Changed lines of the file:
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@@
 	(title_block
 		(title "V2 step")
-		(date "2026-04-14")
+		(date "2026-05-08")
 		(rev "2026-02-10")
 		(company "Versio Duo")
@@
 		(in_pos_files yes)
 		(dnp no)
-		(property "Reference" "#PWR2001"
+		(property "Reference" "#PWR2003"
 			(at 151.13 66.04 0)
 			(hide yes)
@@
 			(project "step"
 				(path "/6c8448b4-b04d-47e1-934e-e40cbe27a7be/2a03ea79-269e-4abf-833c-000ba0ff13d7"
-					(reference "#PWR2001")
+					(reference "#PWR2003")
 					(unit 1)
 				)
@@
 		(in_pos_files yes)
 		(dnp no)
-		(property "Reference" "#PWR2004"
+		(property "Reference" "#PWR2001"
 			(at 138.43 142.24 0)
 			(hide yes)
@@
 			(project "step"
 				(path "/6c8448b4-b04d-47e1-934e-e40cbe27a7be/2a03ea79-269e-4abf-833c-000ba0ff13d7"
-					(reference "#PWR2004")
+					(reference "#PWR2001")
 					(unit 1)
 				)
@@
 		(in_pos_files yes)
 		(dnp no)
-		(property "Reference" "#PWR2003"
+		(property "Reference" "#PWR2004"
 			(at 151.13 106.68 0)
 			(hide yes)
@@
 			(project "step"
 				(path "/6c8448b4-b04d-47e1-934e-e40cbe27a7be/2a03ea79-269e-4abf-833c-000ba0ff13d7"
-					(reference "#PWR2003")
+					(reference "#PWR2004")
 					(unit 1)
 				)
@@
 		(in_pos_files yes)
 		(dnp no)
-		(property "Reference" "#PWR2002"
+		(property "Reference" "#PWR2007"
 			(at 172.72 73.66 0)
 			(hide yes)
@@
 			(project "step"
 				(path "/6c8448b4-b04d-47e1-934e-e40cbe27a7be/2a03ea79-269e-4abf-833c-000ba0ff13d7"
-					(reference "#PWR2002")
+					(reference "#PWR2007")
 					(unit 1)
 				)
@@
 	)
 	(symbol
-		(lib_id "V2_Resistor:0603_100R")
+		(lib_id "V2_Resistor:1608_100R")
 		(at 162.56 80.01 0)
 		(unit 1)
@@
 		(dnp no)
 		(property "Reference" "R2001"
-			(at 167.64 78.74 0)
+			(at 167.386 78.994 0)
 			(show_name no)
 			(do_not_autoplace no)
@@
 		)
 		(property "Value" "100R"
-			(at 166.37 81.28 0)
-			(show_name no)
-			(do_not_autoplace no)
-			(effects
-				(font
-					(size 1.27 1.27)
-				)
-			)
-		)
-		(property "Footprint" "V2_Resistor_SMD:R_0603"
+			(at 166.878 81.28 0)
+			(show_name no)
+			(do_not_autoplace no)
+			(effects
+				(font
+					(size 1.27 1.27)
+				)
+			)
+		)
+		(property "Footprint" "V2_Resistor_SMD:R_1608"
 			(at 162.56 95.758 0)
 			(hide yes)
@@
 		(in_pos_files yes)
 		(dnp no)
-		(property "Reference" "#PWR2007"
+		(property "Reference" "#PWR2006"
 			(at 163.83 147.32 0)
 			(hide yes)
@@
 			(project "step"
 				(path "/6c8448b4-b04d-47e1-934e-e40cbe27a7be/2a03ea79-269e-4abf-833c-000ba0ff13d7"
-					(reference "#PWR2007")
+					(reference "#PWR2006")
 					(unit 1)
 				)
@@
 	)
 	(symbol
-		(lib_id "V2_Capacitor:0603_0u1")
+		(lib_id "V2_Capacitor:1608_0u1")
 		(at 172.72 64.77 0)
 		(unit 1)
@@
 			)
 		)
-		(property "Footprint" "V2_Capacitor_SMD:C_0603"
+		(property "Footprint" "V2_Capacitor_SMD:C_1608"
 			(at 172.72 81.788 0)
 			(hide yes)
@@
 		(in_pos_files yes)
 		(dnp no)
-		(property "Reference" "#PWR2006"
+		(property "Reference" "#PWR2002"
 			(at 148.59 147.32 0)
 			(hide yes)
@@
 			(project "step"
 				(path "/6c8448b4-b04d-47e1-934e-e40cbe27a7be/2a03ea79-269e-4abf-833c-000ba0ff13d7"
-					(reference "#PWR2006")
+					(reference "#PWR2002")
 					(unit 1)
 				)
