File: hardware/step.kicad_pcb (KiCad board)
At the start: 4 copper layers, 150 x 35 mm, 127 parts, among them J101 WAGO 2065-100, J102 WAGO 2065-100, J103 Cortex, J1901 2x05_Horizontal, J2001 2x05_Horizontal, J201 WAGO 2065-100, J202 WAGO 2065-100, J203 WAGO 2065-100, J204 WAGO 2065-100, J301 WAGO 2065-100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

Commit message: Refresh
Parts:
- U201, U301, U401, U501: footprint V2_Package_DFN_QFN:QFN36-5X6 -> V2_Package_DFN_QFN:QFN-36-5X6

Commit message: KiCad 10
Routing:
- net /Enable: track 123.1 -> 103.6 mm

Commit message: Update
Connections:
- net /VDDCORE renamed /+VCORE
