File: hardware/LinkPlug.kicad_sch (KiCad schematic)
At the start: 4 parts, among them J1901 2x05_Horizontal, U1901 THVD2442

Commit message: Update
Parts:
- C1901: Id (none) -> Capacitor:${SYMBOL_NAME}
- J1901: Id (none) -> Header:${SYMBOL_NAME}
- R1901: Id (none) -> Resistor:${SYMBOL_NAME}
- U1901: Id (none) -> RS485:${SYMBOL_NAME}; Rating (none) -> 20Mbps
Other:
- title: V2 Link -> V2 step
Changed lines of the file:
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@@
 	(paper "A4")
 	(title_block
-		(title "V2 Link")
-		(date "2026-03-20")
+		(title "V2 step")
+		(date "2026-04-11")
 		(rev "2026-02-10")
 		(company "Versio Duo")
+		(comment 1 "Stepper Motor Controller")
 	)
 	(rectangle
@@
 			)
 		)
+		(property "Id" "RS485:${SYMBOL_NAME}"
+			(at 146.05 107.95 0)
+			(hide yes)
+			(show_name no)
+			(do_not_autoplace no)
+			(effects
+				(font
+					(size 1.27 1.27)
+				)
+			)
+		)
+		(property "Rating" "20Mbps"
+			(at 147.32 115.57 0)
+			(hide yes)
+			(show_name no)
+			(do_not_autoplace no)
+			(effects
+				(font
+					(size 1.27 1.27)
+				)
+			)
+		)
 		(pin "1"
 		)
@@
 			)
 		)
+		(property "Id" "Resistor:${SYMBOL_NAME}"
+			(at 157.48 85.09 0)
+			(hide yes)
+			(show_name no)
+			(do_not_autoplace no)
+			(effects
+				(font
+					(size 1.27 1.27)
+				)
+			)
+		)
 		(pin "1"
 		)
@@
 			)
 		)
+		(property "Id" "Header:${SYMBOL_NAME}"
+			(at 147.32 147.32 0)
+			(hide yes)
+			(show_name no)
+			(do_not_autoplace no)
+			(effects
+				(font
+					(size 1.27 1.27)
+				)
+			)
+		)
 		(pin "1"
 		)
@@
 			(hide yes)
 			(show_name no)
+			(do_not_autoplace no)
+			(effects
+				(font
+					(size 1.27 1.27)
+				)
+			)
+		)
+		(property "Id" "Capacitor:${SYMBOL_NAME}"
+			(at 166.37 71.12 0)
+			(hide yes)
+			(show_name no)

Commit message: Update
Parts:
- J1901: Rating (none) -> 1A
Changed lines of the file:
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@@
 	(title_block
 		(title "V2 step")
-		(date "2026-04-11")
+		(date "2026-04-14")
 		(rev "2026-02-10")
 		(company "Versio Duo")
@@
 			(hide yes)
 			(show_name no)
+			(do_not_autoplace no)
+			(effects
+				(font
+					(size 1.27 1.27)
+				)
+			)
+		)
+		(property "Rating" "1A"
+			(at 147.32 162.56 0)
+			(hide yes)
+			(show_name no)

Commit message: Good Bye Imperial
Parts:
- C1901: footprint V2_Capacitor_SMD:C_0603 -> V2_Capacitor_SMD:C_1608; symbol V2_Capacitor:0603_0u1 -> V2_Capacitor:1608_0u1
- R1901: footprint V2_Resistor_SMD:R_0603 -> V2_Resistor_SMD:R_1608; symbol V2_Resistor:0603_100R -> V2_Resistor:1608_100R
Changed lines of the file:
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@@
 	(title_block
 		(title "V2 step")
-		(date "2026-04-14")
+		(date "2026-05-08")
 		(rev "2026-02-10")
 		(company "Versio Duo")
@@
 		(in_pos_files yes)
 		(dnp no)
-		(property "Reference" "#PWR1902"
+		(property "Reference" "#PWR1908"
 			(at 166.37 64.77 0)
 			(hide yes)
@@
 			(project "step"
 				(path "/6c8448b4-b04d-47e1-934e-e40cbe27a7be/c6db2f80-f80f-4104-8ca1-02f0ab85cfea"
-					(reference "#PWR1902")
+					(reference "#PWR1908")
 					(unit 1)
 				)
@@
 	)
 	(symbol
-		(lib_id "V2_Resistor:0603_100R")
+		(lib_id "V2_Resistor:1608_100R")
 		(at 157.48 71.12 0)
 		(unit 1)
@@
 		(dnp no)
 		(property "Reference" "R1901"
-			(at 162.56 69.85 0)
+			(at 162.306 69.85 0)
 			(show_name no)
 			(do_not_autoplace no)
@@
 		)
 		(property "Value" "100R"
-			(at 161.29 72.39 0)
-			(show_name no)
-			(do_not_autoplace no)
-			(effects
-				(font
-					(size 1.27 1.27)
-				)
-			)
-		)
-		(property "Footprint" "V2_Resistor_SMD:R_0603"
+			(at 161.798 72.39 0)
+			(show_name no)
+			(do_not_autoplace no)
+			(effects
+				(font
+					(size 1.27 1.27)
+				)
+			)
+		)
+		(property "Footprint" "V2_Resistor_SMD:R_1608"
 			(at 157.48 86.868 0)
 			(hide yes)
@@
 		(in_pos_files yes)
 		(dnp no)
-		(property "Reference" "#PWR1908"
+		(property "Reference" "#PWR1903"
 			(at 148.59 154.94 0)
 			(hide yes)
@@
 			(project "step"
 				(path "/6c8448b4-b04d-47e1-934e-e40cbe27a7be/c6db2f80-f80f-4104-8ca1-02f0ab85cfea"
-					(reference "#PWR1908")
+					(reference "#PWR1903")
 					(unit 1)
 				)
@@
 		(in_pos_files yes)
 		(dnp no)
-		(property "Reference" "#PWR1904"
+		(property "Reference" "#PWR1901"
 			(at 134.62 129.54 0)
 			(hide yes)
@@
 			(project "step"
 				(path "/6c8448b4-b04d-47e1-934e-e40cbe27a7be/c6db2f80-f80f-4104-8ca1-02f0ab85cfea"
-					(reference "#PWR1904")
+					(reference "#PWR1901")
 					(unit 1)
 				)
@@
 		(in_pos_files yes)
 		(dnp no)
-		(property "Reference" "#PWR1906"
+		(property "Reference" "#PWR1902"
 			(at 144.78 134.62 0)
 			(hide yes)
@@
 			(project "step"
 				(path "/6c8448b4-b04d-47e1-934e-e40cbe27a7be/c6db2f80-f80f-4104-8ca1-02f0ab85cfea"
-					(reference "#PWR1906")
+					(reference "#PWR1902")
 					(unit 1)
 				)
@@
 		(in_pos_files yes)
 		(dnp no)
-		(property "Reference" "#PWR1903"
+		(property "Reference" "#PWR1905"
 			(at 146.05 97.79 0)
 			(hide yes)
@@
 			(project "step"
 				(path "/6c8448b4-b04d-47e1-934e-e40cbe27a7be/c6db2f80-f80f-4104-8ca1-02f0ab85cfea"
-					(reference "#PWR1903")
+					(reference "#PWR1905")
 					(unit 1)
 				)
@@
 		(in_pos_files yes)
 		(dnp no)
-		(property "Reference" "#PWR1905"
+		(property "Reference" "#PWR1906"
 			(at 149.86 129.54 0)
 			(hide yes)
@@
 			(project "step"
 				(path "/6c8448b4-b04d-47e1-934e-e40cbe27a7be/c6db2f80-f80f-4104-8ca1-02f0ab85cfea"
-					(reference "#PWR1905")
+					(reference "#PWR1906")
 					(unit 1)
 				)
@@
 		(in_pos_files yes)
 		(dnp no)
-		(property "Reference" "#PWR1901"
+		(property "Reference" "#PWR1904"
 			(at 146.05 57.15 0)
 			(hide yes)
@@
 			(project "step"
 				(path "/6c8448b4-b04d-47e1-934e-e40cbe27a7be/c6db2f80-f80f-4104-8ca1-02f0ab85cfea"
-					(reference "#PWR1901")
+					(reference "#PWR1904")
 					(unit 1)
 				)
@@
 	)
 	(symbol
-		(lib_id "V2_Capacitor:0603_0u1")
+		(lib_id "V2_Capacitor:1608_0u1")
 		(at 166.37 55.88 0)
 		(unit 1)
@@
 			)
 		)
-		(property "Footprint" "V2_Capacitor_SMD:C_0603"
+		(property "Footprint" "V2_Capacitor_SMD:C_1608"
 			(at 166.37 72.898 0)
 			(hide yes)
